File: Elettronica/Schemi/Lab3/circuito_1.sch (KiCad schematic (older format))
At the start: 6 parts

Commit message: Schemi modificati
Parts:
- removed 50~Ohm: Rt, ~, symbol RESISTORE
- renumbered 2~V to 2, 50~Ohm to 50
Connections:
- net at 50.~ (VC): now also GND?.~
Changed lines of the file:
@@
-EESchema Schematic File Version 2  date ven 08 nov 2013 12:14:00 CET
+EESchema Schematic File Version 2  date ven 08 nov 2013 11:15:27 CET
 LIBS:power
 LIBS:device
@@
 $EndDescr
 Wire Wire Line
-	5050 3900 5200 3900
+	6750 4350 5850 4350
 Wire Wire Line
 	6750 4350 6750 4100
 Connection ~ 6300 4350
 Wire Wire Line
-	6950 3900 7250 3900
+	5200 3900 5200 4050
 Wire Wire Line
-	5850 4100 5850 4350
-Wire Wire Line
-	5850 4350 7250 4350
-Connection ~ 6750 4350
+	5850 4350 5850 4100
 Text Notes 5600 3850 0    60   ~ 0
 VB
@@
 $EndComp
 $Comp
-L RESISTORE 50~Ohm
-U 1 1 527CB763
-P 7250 4150
-F 0 "50 Ohm" V 7125 4150 60  0000 C CNN
-F 1 "Rt" V 7375 4150 60  0000 C CNN
-F 2 "~" H 7250 4200 60  0000 C CNN
-F 3 "~" H 7250 4200 60  0000 C CNN
-	1    7250 4150
-	-1   0    0    -1
-$EndComp
-$Comp
 L TERRA GND?
 U 1 1 527CB749
-P 5050 4400
-F 0 "GND?" H 5350 4400 60  0001 C CNN
-F 1 "TERRA" H 5050 4400 60  0001 C CNN
-F 2 "~" H 5050 4400 60  0000 C CNN
-F 3 "~" H 5050 4400 60  0000 C CNN
-	1    5050 4400
+P 5200 4550
+F 0 "GND?" H 5500 4550 60  0001 C CNN
+F 1 "TERRA" H 5200 4550 60  0001 C CNN
+F 2 "~" H 5200 4550 60  0000 C CNN
+F 3 "~" H 5200 4550 60  0000 C CNN
+	1    5200 4550
 	1    0    0    -1
 $EndComp
 $Comp
-L CAVO_COASSIALE_LUNGO 50~Ohm
+L CAVO_COASSIALE_LUNGO 50
 U 1 1 527CB729
 P 6250 3900
@@
 $EndComp
 $Comp
-L GENERATORE_DI_ONDA_QUADRA 2~V
+L GENERATORE_DI_ONDA_QUADRA 2
 U 1 1 527CB719
-P 5050 4100
-F 0 "2 V" V 4900 4100 60  0000 C CNN
-F 1 "GENERATORE_DI_ONDA_QUADRA" H 5050 4100 60  0001 C CNN
-F 2 "~" H 5050 4100 60  0000 C CNN
-F 3 "200 KHz" V 5230 4100 40  0000 C CNN
-	1    5050 4100
+P 5200 4250
+F 0 "2 V" V 5050 4250 60  0000 C CNN
+F 1 "GENERATORE_DI_ONDA_QUADRA" H 5200 4250 60  0001 C CNN
+F 2 "~" H 5200 4250 60  0000 C CNN
+F 3 "200 KHz" V 5380 4250 40  0000 C CNN
+	1    5200 4250
 	1    0    0    -1
 $EndComp
