File: Elettronica/Schemi/Lab3/circuito_2.sch (KiCad schematic (older format))
At the start: 5 parts

Commit message: Schemi modificati
Parts:
- added 100: RESISTORE, ~, symbol RESISTORE
- added 50: 100 Ohm, ~, symbol RESISTORE
- renumbered 2 to 2~V, 50 to 50~Ohm
Connections:
- net at 50~Ohm.~ (VC): now also R?.2
- net at 50~Ohm.~ (VC), GND?.~: now also 100.3, 50.3
- new net: 100.2, 50.2, 50~Ohm.~ (VC)
Changed lines of the file:
@@
-EESchema Schematic File Version 2  date ven 08 nov 2013 11:15:27 CET
+EESchema Schematic File Version 2  date mer 13 nov 2013 10:55:51 CET
 LIBS:power
 LIBS:device
@@
 Sheet 1 1
 Title ""
-Date "8 nov 2013"
+Date "13 nov 2013"
 Rev ""
 Comp ""
@@
 Comment4 ""
 $EndDescr
+Connection ~ 7250 3900
 Wire Wire Line
-	6750 4350 5850 4350
+	7500 3900 6950 3900
+Wire Wire Line
+	7500 4350 5850 4350
+Connection ~ 6750 4350
+Wire Wire Line
+	5850 4350 5850 4100
+Connection ~ 6300 4350
 Wire Wire Line
 	6750 4350 6750 4100
-Connection ~ 6300 4350
 Wire Wire Line
-	5200 3900 5200 4050
-Wire Wire Line
-	5850 4350 5850 4100
+	5050 3900 5200 3900
+Connection ~ 7250 4350
+$Comp
+L RESISTORE 100
+U 1 1 52834C14
+P 7500 4150
+F 0 "100 Ohm" V 7400 4150 50  0000 C CNN
+F 1 "RESISTORE" H 7500 4200 60  0001 C CNN
+F 2 "~" H 7500 4200 60  0000 C CNN
+F 3 "~" H 7500 4200 60  0000 C CNN
+	1    7500 4150
+	1    0    0    -1
+$EndComp
 Text Notes 5600 3850 0    60   ~ 0
 VB
@@
 $EndComp
 $Comp
+L RESISTORE 50
+U 1 1 527CB763
+P 7250 4150
+F 0 "50" H 7125 4150 60  0001 C CNN
+F 1 "100 Ohm" V 7375 4150 50  0000 C CNN
+F 2 "~" H 7250 4200 60  0000 C CNN
+F 3 "~" H 7250 4200 60  0000 C CNN
+	1    7250 4150
+	-1   0    0    -1
+$EndComp
+$Comp
 L TERRA GND?
 U 1 1 527CB749
-P 5200 4550
-F 0 "GND?" H 5500 4550 60  0001 C CNN
-F 1 "TERRA" H 5200 4550 60  0001 C CNN
-F 2 "~" H 5200 4550 60  0000 C CNN
-F 3 "~" H 5200 4550 60  0000 C CNN
-	1    5200 4550
+P 5050 4400
+F 0 "GND?" H 5350 4400 60  0001 C CNN
+F 1 "TERRA" H 5050 4400 60  0001 C CNN
+F 2 "~" H 5050 4400 60  0000 C CNN
+F 3 "~" H 5050 4400 60  0000 C CNN
+	1    5050 4400
 	1    0    0    -1
 $EndComp
 $Comp
-L CAVO_COASSIALE_LUNGO 50
+L CAVO_COASSIALE_LUNGO 50~Ohm
 U 1 1 527CB729
 P 6250 3900
@@
 $EndComp
 $Comp
-L GENERATORE_DI_ONDA_QUADRA 2
+L GENERATORE_DI_ONDA_QUADRA 2~V
 U 1 1 527CB719
-P 5200 4250
-F 0 "2 V" V 5050 4250 60  0000 C CNN
-F 1 "GENERATORE_DI_ONDA_QUADRA" H 5200 4250 60  0001 C CNN
-F 2 "~" H 5200 4250 60  0000 C CNN
-F 3 "200 KHz" V 5380 4250 40  0000 C CNN
-	1    5200 4250
+P 5050 4100
+F 0 "2 V" V 4900 4100 60  0000 C CNN
+F 1 "GENERATORE_DI_ONDA_QUADRA" H 5050 4100 60  0001 C CNN
+F 2 "~" H 5050 4100 60  0000 C CNN
+F 3 "200 KHz" V 5230 4100 40  0000 C CNN
+	1    5050 4100
 	1    0    0    -1
 $EndComp
